File: Breakout-68040/Breakout-68040.kicad_pcb (KiCad board)
At the start: 4 copper layers, 100 x 100 mm, 49 parts, among them IC1 DS1232S+, IC2 ATF22V10C-7PU, J1 Conn_02x32_Odd_Even, J10 Conn_01x03_Pin, J2 Conn_01x02_Pin, J3 Conn_01x32_Pin, J4 Conn_02x32_Odd_Even, J5 Conn_02x16_Odd_Even, J6 Conn_01x16_Pin, J7 Conn_01x08_Pin, J8 Conn_02x12_Odd_Even, J9 Conn_01x03_Pin, SW1 Reset, U1 MC680LC40, X1 SG-615

Commit message: Mothballing
Connections:
- IC2 pad 1: CLK/IN -> PCLK
- IC2 pad 22: PCLK -> I/O_9
- J8 pad 1: CLK/IN -> PCLK
- J8 pad 6: PCLK -> I/O_9
Routing:
- net I/O_9: track 0.00 -> 12.9 mm
- net PCLK: track 66.0 -> 56.2 mm, vias 1 -> 0
- net CLK/IN: track 7.99 -> 0.00 mm
Changed lines of the file:
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@@
 	(net 128 "I{slash}O_7")
 	(net 129 "IN_3")
-	(net 130 "CLK{slash}IN")
+	(net 130 "I{slash}O_9")
 	(net 131 "I{slash}O_3")
 	(net 132 "IN_6")
@@
 		(tags "Through hole pin header THT 2x12 2.54mm double row")
 		(property "Reference" "J8"
-			(at 1.27 -2.33 -90)
+			(at 0.15 -2.1 -90)
 			(layer "F.SilkS")
 			(effects
@@
 			(layers "*.Cu" "*.Mask")
 			(remove_unused_layers no)
-			(net 130 "CLK{slash}IN")
+			(net 111 "PCLK")
 			(pinfunction "Pin_1")
 			(pintype "passive")
@@
 			(layers "*.Cu" "*.Mask")
 			(remove_unused_layers no)
-			(net 111 "PCLK")
+			(net 130 "I{slash}O_9")
 			(pinfunction "Pin_6")
 			(pintype "passive")
@@
 		(tags "capacitor handsolder")
 		(property "Reference" "C1"
-			(at 0 -1.68 270)
+			(at 0 -1.68 -90)
 			(layer "F.SilkS")
 			(hide yes)
@@
 		)
 		(property "Value" "100nF"
-			(at 0 1.68 270)
+			(at 0 1.68 -90)
 			(layer "F.Fab")
 			(hide yes)
@@
 		)
 		(fp_text user "${REFERENCE}"
-			(at 0 0 270)
+			(at 0 0 -90)
 			(layer "F.Fab")
 			(effects
@@
 			(layers "*.Cu" "*.Mask")
 			(remove_unused_layers no)
-			(net 130 "CLK{slash}IN")
+			(net 111 "PCLK")
 			(pinfunction "CLK/IN")
 			(pintype "passive")
@@
 			(layers "*.Cu" "*.Mask")
 			(remove_unused_layers no)
-			(net 111 "PCLK")
+			(net 130 "I{slash}O_9")
 			(pinfunction "I/O_9")
 			(pintype "passive")
@@
 		(layer "Edge.Cuts")
 	)
-	(gr_text "GND"
-		(at 117.6 135.2 0)
-		(layer "In1.Cu")
-		(effects
-			(font
-				(size 1 1)
-				(thickness 0.15)
-			)
-			(justify left bottom)
-		)
-	)
-	(gr_text "+5V"
-		(at 117.6 132.4 0)
-		(layer "In1.Cu")
-		(effects
-			(font
-				(size 1 1)
-				(thickness 0.15)
-			)
-			(justify left bottom)
-		)
-	)
 	(gr_text "TM1"
 		(at 107.283852 140.435 90)
@@
 		)
 	)
+	(gr_text "+5V"
+		(at 118 132.5 0)
+		(layer "F.SilkS")
+		(effects
+			(font
+				(size 1 1)
+				(thickness 0.1)
+			)
+			(justify left bottom)
+		)
+	)
 	(gr_text "A5"
 		(at 28.1 128.218482 0)
@@
 	)
 	(gr_text "1200ms"
-		(at 96.4 112 0)
+		(at 96.4 112.5 0)
 		(layer "F.SilkS")
 		(effects
@@
 		)
 	)
+	(gr_text "GND"
+		(at 118 135.25 0)
+		(layer "F.SilkS")
+		(effects
+			(font
+				(size 1 1)
+				(thickness 0.1)
+			)
+			(justify left bottom)
+		)
+	)
 	(gr_text "A8"
 		(at 28.1 120.60558 0)
@@
 	)
 	(segment
-		(start 56.11 120.8)
-		(end 58.005 118.905)
-		(width 0.25)
-		(locked yes)
-		(layer "F.Cu")
-		(net 111)
-	)
-	(segment
 		(start 56.7425 106.698)
 		(end 56.155 107.285)
@@
 	)
 	(segment
-		(start 51.9 120.8)
-		(end 56.11 120.8)
+		(start 54.4933 107.285)
+		(end 53.615 108.163)
 		(width 0.25)
 		(locked yes)
@@
 	)
 	(segment
-		(start 57.8122 132.0367)
-		(end 57.0033 132.8456)
-		(width 0.25)
-		(layer "F.Cu")
-		(net 111)
-	)
-	(segment
-		(start 54.4933 107.285)
-		(end 53.615 108.163)
+		(start 52.925 126.525)
+		(end 44.185 126.525)
 		(width 0.25)
 		(locked yes)
@@
 	)
 	(segment
-		(start 50.32 119.22)
-		(end 51.9 120.8)
-		(width 0.25)
-		(locked yes)
-		(layer "F.Cu")
-		(net 111)
-	)
-	(segment
 		(start 53.5725 115.968)
 		(end 53.615 115.9255)
@@
 	)
 	(segment
-		(start 57.0033 132.8456)
-		(end 57.0033 133.7205)
-		(width 0.25)
-		(layer "F.Cu")
-		(net 111)
-	)
-	(segment
-		(start 58.18 130.86)
-		(end 58.18 132.0367)
-		(width 0.25)
-		(layer "F.Cu")
-		(net 111)
-	)
-	(segment
-		(start 57.0033 133.7205)
-		(end 54.6564 136.0674)
-		(width 0.25)
-		(layer "F.Cu")
-		(net 111)
-	)
-	(segment
-		(start 58.18 132.0367)
-		(end 57.8122 132.0367)
+		(start 44.185 126.525)
+		(end 43.6 125.94)
 		(width 0.25)
 		(layer "F.Cu")
@@
 	)
 	(segment
-		(start 54.6564 136.0674)
-		(end 53.8963 136.0674)
-		(width 0.25)
-		(layer "F.Cu")
-		(net 111)
-	)
-	(segment
 		(start 50.32 119.22)
 		(end 48.32 121.22)
@@
 		(net 111)
 	)
-	(via
-		(at 53.8963 136.0674)
-		(size 0.7)
-		(drill 0.3)
-		(layers "F.Cu" "B.Cu")
+	(segment
+		(start 51.9233 131.4144)
+		(end 52.7322 132.2233)
+		(width 0.25)
+		(layer "B.Cu")
 		(net 111)
 	)
 	(segment
-		(start 48.46 141.6833)
-		(end 53.8963 136.247)
+		(start 51.9233 129.0534)
+		(end 51.9233 131.4144)
 		(width 0.25)
 		(layer "B.Cu")
@@
 	)
 	(segment
-		(start 53.8963 136.247)
-		(end 53.8963 136.0674)
+		(start 53.1 133.4)
+		(end 53.1 137.0433)
 		(width 0.25)
 		(layer "B.Cu")
@@
 	)
 	(segment
-		(start 58.005 118.905)
-		(end 58.005 120.4317)
+		(start 48.46 141.6833)
+		(end 48.57165 141.57165)
 		(width 0.25)
 		(layer "B.Cu")
@@
 	)
 	(segment
-		(start 58.18 130.86)
-		(end 58.18 129.6833)
+		(start 53.1 137.0433)
+		(end 48.57165 141.57165)
 		(width 0.25)
 		(layer "B.Cu")
@@
 	)
 	(segment
-		(start 59.1794 121.6061)
-		(end 59.1794 128.6839)
+		(start 52.7322 132.2233)
+		(end 53.1 132.2233)
 		(width 0.25)
 		(layer "B.Cu")
@@
 	)
 	(segment
-		(start 58.005 120.4317)
-		(end 59.1794 121.6061)
+		(start 53.1 133.4)
+		(end 53.1 132.2233)
 		(width 0.25)
 		(layer "B.Cu")
@@
 	)
 	(segment
-		(start 59.1794 128.6839)
-		(end 58.18 129.6833)
+		(start 52.925 128.0517)
+		(end 51.9233 129.0534)
+		(width 0.25)
+		(layer "B.Cu")
+		(net 111)
+	)
+	(segment
+		(start 52.925 126.525)
+		(end 52.925 128.0517)
 		(width 0.25)
 		(layer "B.Cu")
@@
 	)
 	(segment
-		(start 51.9233 131.4144)
-		(end 52.7322 132.2233)
-		(width 0.25)
-		(layer "B.Cu")
-		(net 130)
-	)
-	(segment
-		(start 51.9233 129.0534)
-		(end 51.9233 131.4144)
+		(start 58.005 118.905)
+		(end 58.005 120.4317)
 		(width 0.25)
 		(layer "B.Cu")
@@
 	)
 	(segment
-		(start 52.7322 132.2233)
-		(end 53.1 132.2233)
+		(start 58.18 130.86)
+		(end 58.18 129.6833)
 		(width 0.25)
 		(layer "B.Cu")
@@
 	)
 	(segment
-		(start 53.1 133.4)
-		(end 53.1 132.2233)
+		(start 59.1794 121.6061)
+		(end 59.1794 128.6839)
 		(width 0.25)
 		(layer "B.Cu")
@@
 	)
 	(segment
-		(start 52.925 128.0517)
-		(end 51.9233 129.0534)
+		(start 58.005 120.4317)
+		(end 59.1794 121.6061)
 		(width 0.25)
 		(layer "B.Cu")
@@
 	)
 	(segment
-		(start 52.925 126.525)
-		(end 52.925 128.0517)
+		(start 59.1794 128.6839)
+		(end 58.18 129.6833)
 		(width 0.25)
 		(layer "B.Cu")
