File: Breakout-68040/Breakout-68040.kicad_sch (KiCad schematic)
At the start: 14 parts, among them J1 Conn_02x32_Odd_Even, J2 Conn_01x04_Pin, J3 Conn_01x32_Pin, J4 Conn_02x32_Odd_Even, J5 Conn_02x16_Odd_Even, U1 MC680LC40

Commit message: First commit
Parts:
- removed D1, D2, D3, D4: LED, symbol Device:LED
- removed J2: Conn_01x04_Pin, Connector_PinHeader_1.27mm:PinHeader_1x04_P1.27mm_Vertical, symbol Connector:Conn_01x04_Pin
- removed R1, R2, R3, R4: 1K, Resistor_THT:R_Axial_DIN0207_L6.3mm_D2.5mm_P10.16mm_Horizontal, symbol Device:R
- added C1, C10, C11, C12, C13, C14, C15, C16, C17, C18, C19, C2, C20, C21, C22, C23, C24, C25, C26, C27, C28, C29, C3, C30, C4, C5, C6, C7, C8, C9: 100uF, Capacitor_SMD:C_0603_1608Metric_Pad1.08x0.95mm_HandSolder, symbol Device:C
- added D10, D11, D12, D5, D6, D7, D8, D9: LED, LED_SMD:LED_0603_1608Metric_Pad1.05x0.95mm_HandSolder, symbol Device:LED
- added IC1: DS1232S+, Package_SO:SOIC-16W_7.5x10.3mm_P1.27mm, symbol DS1232S:DS1232S+
- added IC2: ATF22V10C-7PU, Package_DIP:DIP-24_W7.62mm_LongPads, symbol ATF22V10:ATF22V10C-15PU
- added J6: Conn_01x16_Pin, Connector_PinHeader_2.54mm:PinHeader_1x16_P2.54mm_Vertical, symbol Connector:Conn_01x16_Pin
- added J7: Conn_01x08_Pin, Connector_PinHeader_2.54mm:PinHeader_1x08_P2.54mm_Vertical, symbol Connector:Conn_01x08_Pin
- added J8: Conn_02x12_Odd_Even, Connector_PinHeader_2.54mm:PinHeader_2x12_P2.54mm_Vertical, symbol Connector_Generic:Conn_02x12_Odd_Even
- added R10, R11, R12, R5, R6, R7, R8, R9: 1K, Resistor_SMD:R_0603_1608Metric_Pad0.98x0.95mm_HandSolder, symbol Device:R
- added SW1: Reset, Button_Switch_THT:SW_TH_Tactile_Omron_B3F-10xx, symbol Switch:SW_Push
- added X1: SG-615, Oscillator:Oscillator_SMD_SeikoEpson_SG8002JA-4Pin_14.0x8.7mm, symbol Oscillator:SG-615
Connections:
- net BCLK: now also J4.51 (Pin_51), IC2.23 (I/O_10), J8.4 (Pin_4); no longer J5.17 (Pin_17)
- net GND: now also U1.B02 (GND_B02), U1.B04 (GND_B04), U1.B06 (GND_B06), U1.B08 (GND_B08), U1.B10 (GND_B10), U1.B13 (GND_B13), U1.B15 (GND_B15), U1.B17 (GND_B17), U1.C06 (GND_C06), U1.C07 (GND_C07), U1.C09 (GND_C09), U1.C11 (GND_C11), U1.C13 (GND_C13), U1.D02 (GND_D02), U1.D17 (GND_D17), U1.F02 (GND_F02), U1.F17 (GND_F17), U1.H02 (GND_H02), U1.H17 (GND_H17), U1.K03 (GND_K03), U1.K16 (GND_K16), U1.L02 (GND_L02), U1.L03 (GND_L03), U1.L17 (GND_L17), U1.M16 (GND_M16), U1.N02 (GND_N02), U1.N17 (GND_N17), U1.Q02 (GND_Q02), U1.Q17 (GND_Q17), U1.R04 (GND_R04), U1.R06 (GND_R06), U1.R10 (GND_R10), U1.R11 (GND_R11), U1.R13 (GND_R13), U1.S02 (GND_S02), U1.S09 (GND_S09), U1.S10 (GND_S10), U1.S15 (GND_S15), U1.S17 (GND_S17), U1.T04 (GND_T04), C1.2, C10.2, C11.2, C12.2, C13.2, C14.2, C15.2, C16.2, C17.2, C18.2, C19.2, C2.2, C20.2, C21.2, C22.2, C23.2, C24.2, C25.2, C26.2, C27.2, C28.2, C29.2, C3.2, C30.2, C4.2, C5.2, C6.2, C7.2, C8.2, C9.2, IC1.8 (GND), IC2.12 (GND), R10.2, R11.2, R12.2, R5.2, R6.2, R7.2, R8.2, R9.2, SW1.1, X1.2 (GND)
- net PCLK: now also J4.53 (Pin_53), IC2.22 (I/O_9), J8.6 (Pin_6), X1.3 (OUT); no longer J5.19 (Pin_19)
- net PST0: now also J4.43 (Pin_43); no longer J5.9 (Pin_9)
- net PST1: now also J4.45 (Pin_45); no longer J5.11 (Pin_11)
- net PST2: now also J4.47 (Pin_47); no longer J5.13 (Pin_13)
- net PST3: now also J4.49 (Pin_49); no longer J5.15 (Pin_15)
- net SC0: now also J5.9 (Pin_9); no longer J4.43 (Pin_43)
- net SC1: now also J5.11 (Pin_11); no longer J4.45 (Pin_45)
- net ~{BB}: now also J5.19 (Pin_19); no longer J4.53 (Pin_53)
- net ~{BG}: now also J5.17 (Pin_17); no longer J4.51 (Pin_51)
- net ~{BR}: now also J5.15 (Pin_15); no longer J4.49 (Pin_49)
- net ~{MI}: now also J5.13 (Pin_13); no longer J4.47 (Pin_47)
- net ~{RSTI}: now also IC1.11 (~{RST})
- net ~{TS}: now also IC1.13 (~{ST})
- net +5V: now reaches U1.B05 (VCC_B05)
- net +5V: now also U1.B09 (VCC_B09), U1.B14 (VCC_B14), U1.C02 (VCC_C02), U1.C05 (VCC_C05), U1.C08 (VCC_C08), U1.C10 (VCC_C10), U1.C12 (VCC_C12), U1.C14 (VCC_C14), U1.C17 (VCC_C17), U1.G02 (VCC_G02), U1.G17 (VCC_G17), U1.H03 (VCC_H03), U1.H16 (VCC_H16), U1.J03 (VCC_J03), U1.J16 (VCC_J16), U1.L16 (VCC_L16), U1.M02 (VCC_M02), U1.M03 (VCC_M03), U1.M17 (VCC_M17), U1.R02 (VCC_R02), U1.R05 (VCC_R05), U1.R08 (VCC_R08), U1.R12 (VCC_R12), U1.R17 (VCC_R17), U1.S08 (VCC_S08), U1.S16 (VCC_S16), C1.1, C10.1, C11.1, C12.1, C13.1, C14.1, C15.1, C16.1, C17.1, C18.1, C19.1, C2.1, C20.1, C21.1, C22.1, C23.1, C24.1, C25.1, C26.1, C27.1, C28.1, C29.1, C3.1, C30.1, C4.1, C5.1, C6.1, C7.1, C8.1, C9.1, IC1.15 (VCC), IC1.6 (TOL), IC2.24 (VCC), J6.1 (Pin_1), J6.10 (Pin_10), J6.11 (Pin_11), J6.12 (Pin_12), J6.13 (Pin_13), J6.14 (Pin_14), J6.15 (Pin_15), J6.16 (Pin_16), J6.2 (Pin_2), J6.3 (Pin_3), J6.4 (Pin_4), J6.5 (Pin_5), J6.6 (Pin_6), J6.7 (Pin_7), J6.8 (Pin_8), J6.9 (Pin_9), X1.4 (Vcc)
- new net: D12.1 (K), R12.1
- new net: D11.1 (K), R11.1
- new net: IC1.2 (~{PBRST}), SW1.2
- new net: D10.1 (K), R10.1
- new net: D10.2 (A), J7.6 (Pin_6)
- new net: D6.1 (K), R6.1
- new net: D8.1 (K), R8.1
- new net: D8.2 (A), J7.4 (Pin_4)
- new net: D9.1 (K), R9.1
- new net: D9.2 (A), J7.5 (Pin_5)
- new net: D5.1 (K), R5.1
- new net: D12.2 (A), J7.8 (Pin_8)
- new net: D5.2 (A), J7.1 (Pin_1)
- new net: D6.2 (A), J7.2 (Pin_2)
- new net: D7.2 (A), J7.3 (Pin_3)
- new net: D11.2 (A), J7.7 (Pin_7)
- new net: D7.1 (K), R7.1
- new net CLK/IN: IC2.1 (CLK/IN), J8.1 (Pin_1)
- new net IN_1: IC2.2 (IN_1), J8.3 (Pin_3)
- new net IN_10: IC2.13 (IN_10), J8.24 (Pin_24)
- new net IN_2: IC2.3 (IN_2), J8.5 (Pin_5)
- new net IN_3: IC2.5 (IN_3), J8.9 (Pin_9)
- new net IN_4: IC2.6 (IN_4), J8.11 (Pin_11)
- new net IN_5: IC2.7 (IN_5), J8.13 (Pin_13)
- new net IN_6: IC2.8 (IN_6), J8.15 (Pin_15)
- new net IN_7: IC2.9 (IN_7), J8.17 (Pin_17)
- new net IN_8: IC2.10 (IN_8), J8.19 (Pin_19)
- new net IN_9: IC2.11 (IN_9), J8.21 (Pin_21)
- new net IN/PD: IC2.4 (IN/PD), J8.7 (Pin_7)
- new net I/O_1: IC2.14 (I/O_1), J8.22 (Pin_22)
- new net I/O_2: IC2.15 (I/O_2), J8.20 (Pin_20)
- new net I/O_3: IC2.16 (I/O_3), J8.18 (Pin_18)
- new net I/O_4: IC2.17 (I/O_4), J8.16 (Pin_16)
- new net I/O_5: IC2.18 (I/O_5), J8.14 (Pin_14)
- new net I/O_6: IC2.19 (I/O_6), J8.12 (Pin_12)
- new net I/O_7: IC2.20 (I/O_7), J8.10 (Pin_10)
- new net I/O_8: IC2.21 (I/O_8), J8.8 (Pin_8)
- no-connect marks 0 -> 13
Other:
- note added: "TD not connected = 600ms watchdog timer TOL connected to +5v = 10% tolerance on VCC"

Commit message: First routed version
Parts:
- removed C16, C24, C25, C26, C27, C28, C30, C9: 100uF, Capacitor_SMD:C_0603_1608Metric_Pad1.08x0.95mm_HandSolder, symbol Device:C
- removed D10, D11, D12, D5, D6, D7, D8, D9: LED, LED_SMD:LED_0603_1608Metric_Pad1.05x0.95mm_HandSolder, symbol Device:LED
- removed R10, R11, R12, R5, R6, R7, R8, R9: 1K, Resistor_SMD:R_0603_1608Metric_Pad0.98x0.95mm_HandSolder, symbol Device:R
- added D1: Power LED, LED_SMD:LED_0603_1608Metric_Pad1.05x0.95mm_HandSolder, symbol Device:LED
- added D19, D20, D21, D22, D23, D24, D25, D26: LED, LED_SMD:LED_0805_2012Metric_Pad1.15x1.40mm_HandSolder, symbol Device:LED
- added J10, J9: Conn_01x03_Pin, Connector_PinHeader_2.54mm:PinHeader_1x03_P2.54mm_Vertical, symbol Connector:Conn_01x03_Pin
- added J2: Conn_01x02_Pin, Connector_PinHeader_2.54mm:PinHeader_1x02_P2.54mm_Vertical, symbol Connector:Conn_01x02_Pin
- added R1: 1K, Resistor_SMD:R_0603_1608Metric_Pad0.98x0.95mm_HandSolder, symbol Device:R
- added RN1: 1K, Resistor_SMD:R_Array_Convex_8x0602, symbol Device:R_Pack08
Connections:
- net +5V: now also J10.1 (Pin_1), J2.1 (Pin_1), J9.1 (Pin_1), R1.1; no longer IC1.6 (TOL)
- net GND: now also D1.1 (K), D19.1 (K), D20.1 (K), D21.1 (K), D22.1 (K), D23.1 (K), D24.1 (K), D25.1 (K), D26.1 (K), J10.3 (Pin_3), J2.2 (Pin_2), J9.3 (Pin_3)
- net ~{CDIS}: now also J4.35 (Pin_35); no longer J5.1 (Pin_1)
- net ~{MDIS}: now also J4.41 (Pin_41); no longer J5.7 (Pin_7)
- net ~{RSTI}: now also J4.37 (Pin_37); no longer J5.3 (Pin_3)
- net ~{RSTO}: now also J4.39 (Pin_39); no longer J5.5 (Pin_5)
- net ~{TA}: now also J5.1 (Pin_1); no longer J4.35 (Pin_35)
- net ~{TBI}: now also J5.7 (Pin_7); no longer J4.41 (Pin_41)
- net ~{TCI}: now also J5.5 (Pin_5); no longer J4.39 (Pin_39)
- net ~{TEA}: now also J5.3 (Pin_3); no longer J4.37 (Pin_37)
- net at IC1.4 (TD): now also J9.2 (Pin_2)
- net at J7.6 (Pin_6): now also RN1.14 (R3.2)
- net at J7.4 (Pin_4): now also RN1.12 (R5.2)
- net at J7.5 (Pin_5): now also RN1.13 (R4.2)
- net at J7.8 (Pin_8): now also RN1.16 (R1.2)
- net at J7.1 (Pin_1): now also RN1.9 (R8.2)
- net at J7.2 (Pin_2): now also RN1.10 (R7.2)
- net at J7.3 (Pin_3): now also RN1.11 (R6.2)
- net at J7.7 (Pin_7): now also RN1.15 (R2.2)
- new net: IC1.6 (TOL), J10.2 (Pin_2)
- new net: D21.2 (A), RN1.6 (R6.1)
- new net: D23.2 (A), RN1.4 (R4.1)
- new net: D20.2 (A), RN1.7 (R7.1)
- new net: D22.2 (A), RN1.5 (R5.1)
- new net: D25.2 (A), RN1.2 (R2.1)
- new net: D19.2 (A), RN1.8 (R8.1)
- new net: D26.2 (A), RN1.1 (R1.1)
- new net: D24.2 (A), RN1.3 (R3.1)
- new net: D1.2 (A), R1.2
- no-connect marks 13 -> 12
Other:
- note removed: "TD not connected = 600ms watchdog timer TOL connected to +5v = 10% tolerance on VCC"
- moved on the sheet: C10, C11, C12, C13, C14, C15, C17, C18, C19, C20, C21, C22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

Commit message: JLCPCB manufacturing info
Parts:
- removed C1, C2, C3: 100uF, Capacitor_SMD:C_0603_1608Metric_Pad1.08x0.95mm_HandSolder, symbol Device:C
- removed RN1: 1K, Resistor_SMD:R_Array_Convex_8x0602, symbol Device:R_Pack08
- added RN1: 1K, Resistor_SMD:R_Array_Convex_4x0603, symbol Device:R_Pack04
- added RN2: R_Pack04, Resistor_SMD:R_Array_Convex_4x0603, symbol Device:R_Pack04
- C10, C11, C12, C13, C14, C15, C17, C18, C19, C20, C21, C22, C23, C29, C4, C5, C6, C7, C8: value 100uF -> 100nF; footprint Capacitor_SMD:C_0603_1608Metric_Pad1.08x0.95mm_HandSolder -> Capacitor_SMD:C_0805_2012Metric_Pad1.18x1.45mm_HandSolder; JLC (none) -> 0805; LCSC (none) -> C49678
- D1: footprint LED_SMD:LED_0603_1608Metric_Pad1.05x0.95mm_HandSolder -> LED_SMD:LED_0805_2012Metric_Pad1.15x1.40mm_HandSolder; JLC (none) -> 0805; LCSC (none) -> C2297
- D19, D20, D21, D22, D23, D24, D25, D26: JLC (none) -> 805; LCSC (none) -> C2297
- R1: footprint Resistor_SMD:R_0603_1608Metric_Pad0.98x0.95mm_HandSolder -> Resistor_SMD:R_0805_2012Metric_Pad1.20x1.40mm_HandSolder; JLC (none) -> 805; LCSC (none) -> C17513
Connections:
- net at J7.1 (Pin_1): now also RN1.5 (R4.2)
- net at J7.2 (Pin_2): now also RN1.6 (R3.2)
- net at J7.3 (Pin_3): now also RN1.7 (R2.2)
- net at J7.4 (Pin_4): now also RN1.8 (R1.2)
- net at J7.5 (Pin_5): now also RN2.5 (R4.2)
- net at J7.6 (Pin_6): now also RN2.6 (R3.2)
- net at J7.7 (Pin_7): now also RN2.7 (R2.2)
- net at J7.8 (Pin_8): now also RN2.8 (R1.2)
- net at D21.2 (A): now also RN1.2 (R2.1)
- net at D23.2 (A): now also RN2.4 (R4.1)
- net at D20.2 (A): now also RN1.3 (R3.1)
- net at D22.2 (A): now also RN1.1 (R1.1)
- net at D25.2 (A): now also RN2.2 (R2.1)
- net at D19.2 (A): now also RN1.4 (R4.1)
- net at D26.2 (A): now also RN2.1 (R1.1)
- net at D24.2 (A): now also RN2.3 (R3.1)
Other:
- moved on the sheet: C17, C18, C19, C20, C21, C22, C23, C29

Commit message: Sent to jclpcb
Parts:
- added C1, C2, C3: 100nF, Capacitor_SMD:C_0805_2012Metric_Pad1.18x1.45mm_HandSolder, symbol Device:C
Connections:
- net +5V: now also C1.1, C2.1, C3.1
- net GND: now also C1.2, C2.2, C3.2
Other:
- moved on the sheet: C10, C11, C12, C13, C14, C15, C17, C18, C19, C20, C21, C22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

Commit message: Mothballing
Connections:
- net CLK/IN is gone; now on net PCLK: IC2.1 (CLK/IN), J8.1 (Pin_1)
- net PCLK: no longer IC2.22 (I/O_9), J8.6 (Pin_6)
- new net I/O_9: IC2.22 (I/O_9), J8.6 (Pin_6)
Changed lines of the file:
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@@
 		)
 	)
-	(global_label "PCLK"
+	(global_label "I{slash}O_9"
 		(shape input)
 		(at 195.58 251.46 0)
@@
 		)
 		(property "Intersheetrefs" "${INTERSHEET_REFS}"
-			(at 203.4033 251.46 0)
+			(at 204.0081 251.46 0)
 			(effects
 				(font
@@
 		)
 	)
-	(global_label "PCLK"
+	(global_label "I{slash}O_9"
 		(shape input)
 		(at 238.76 251.46 0)
@@
 		)
 		(property "Intersheetrefs" "${INTERSHEET_REFS}"
-			(at 246.5833 251.46 0)
+			(at 247.1881 251.46 0)
 			(effects
 				(font
@@
 		)
 	)
-	(global_label "CLK{slash}IN"
+	(global_label "PCLK"
 		(shape input)
 		(at 162.56 246.38 180)
@@
 		)
 		(property "Intersheetrefs" "${INTERSHEET_REFS}"
-			(at 152.7409 246.38 0)
+			(at 154.7367 246.38 0)
 			(effects
 				(font
@@
 		)
 	)
-	(global_label "CLK{slash}IN"
+	(global_label "PCLK"
 		(shape input)
 		(at 226.06 246.38 180)
@@
 		)
 		(property "Intersheetrefs" "${INTERSHEET_REFS}"
-			(at 216.2409 246.38 0)
-			(effects
-				(font
+			(at 218.2367 246.38 0)
+			(effects
+				(font
